File: mo5-connector-pcb/mo5-connector-pcb.kicad_pcb (KiCad board)
At the start: 2 copper layers, 50.2 x 53.3 mm, 26 parts

Commit message: Prepare for production
Other:
- board text added: "MO5 Connector Board Groep 10"
Changed lines of the file:
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@@
     (pad_to_mask_clearance 0)
     (pcbplotparams
-      (layerselection 0x00010fc_ffffffff)
+      (layerselection 0x0001000_fffffffe)
       (plot_on_all_layers_selection 0x0000000_00000000)
       (disableapertmacros false)
@@
       (outputformat 1)
       (mirror false)
-      (drillshape 1)
+      (drillshape 0)
       (scaleselection 1)
       (outputdirectory "")
@@
       (net 24 "Net-(A1-D10)") (pinfunction "1") (pintype "input"))
   )
-  (gr_rect (start 175.241976 52.07) (end 125.076976 105.41)
+  (gr_rect (start 125.076976 52.07) (end 175.241976 105.41)
     (stroke (width 0.1) (type default)) (fill none) (layer "Edge.Cuts"))
+  (gr_text "MO5 Connector Board\nGroep 10" (at 148.082 75.311 180) (layer "B.Cu")
+    (effects (font (size 1.5 1.5) (thickness 0.1875)) (justify left bottom mirror))
+  )
   (segment (start 135.998976 62.103) (end 138.498976 62.103) (width 2) (layer "B.Cu") (net 4))
   (segment (start 144.126976 56.475) (end 144.126976 54.61) (width 2) (layer "B.Cu") (net 4))
